Commit message: Add cylinder and gripper friction

File: urdf/object.xacro (robot description, xacro)
@@ -5,5 +5,5 @@
     <visual>
       <geometry>
-        <cylinder radius="0.01" length="0.5"/>
+        <cylinder radius="0.01" length="0.3"/>
       </geometry>
       <material name="blue">
@@ -14,6 +14,22 @@
     <collision>
       <geometry>
-        <cylinder radius="0.01" length="0.5"/>
+        <cylinder radius="0.01" length="0.3"/>
       </geometry>
+      <surface>
+        <friction>
+          <ode>
+            <mu>100.0</mu>
+            <mu2>100.0</mu2>
+          </ode>
+        </friction>
+        <contact>
+          <ode>
+            <kp>1000.0</kp>
+            <kd>1.0</kd>
+            <max_vel>0.1</max_vel>
+            <min_depth>0.01</min_depth>
+          </ode>
+        </contact>
+      </surface>
     </collision>
     <!-- Inertial for dynamics -->
@@ -22,8 +38,8 @@
       <origin xyz="0 0 0" rpy="0 0 0"/>
       <inertia
-        ixx="0.0001"
+        ixx="0.001"
         ixy="0.0"
         ixz="0.0"
-        iyy="0.0001"
+        iyy="0.001"
         iyz="0.0"
         izz="0.0001"/>

File: urdf/ur_macro.xacro (robot description, xacro)
@@ -538,4 +538,20 @@
           <mesh filename="file://$(find my_ur)/meshes/robotiq_85_gripper/collision/robotiq_85_finger_link.stl"/>
         </geometry>
+        <surface>
+          <friction>
+            <ode>
+              <mu>100.0</mu>
+              <mu2>100.0</mu2>
+            </ode>
+          </friction>
+          <contact>
+            <ode>
+              <kp>10000.0</kp>
+              <kd>1.0</kd>
+              <max_vel>0.1</max_vel>
+              <min_depth>0.001</min_depth>
+            </ode>
+          </contact>
+        </surface>
       </collision>
       <inertial>
@@ -557,4 +573,20 @@
           <mesh filename="file://$(find my_ur)/meshes/robotiq_85_gripper/collision/robotiq_85_finger_link.stl"/>
         </geometry>
+        <surface>
+          <friction>
+            <ode>
+              <mu>100.0</mu>
+              <mu2>100.0</mu2>
+            </ode>
+          </friction>
+          <contact>
+            <ode>
+              <kp>10000.0</kp>
+              <kd>1.0</kd>
+              <max_vel>0.1</max_vel>
+              <min_depth>0.001</min_depth>
+            </ode>
+          </contact>
+        </surface>
       </collision>
       <inertial>
