Commit message: A bunch of bug fixes

File: urdf/gripper.urdf.xacro (robot description, xacro)
@@ -34,5 +34,4 @@
       <origin rpy="0.0 0.0 0.0" xyz="0.05490451627 -0.03060114443 0.0"/>
       <limit lower="-3.14" upper="3.14" velocity="3.14" effort="1000"/>
-      <mimic joint="robotiq_85_left_knuckle_joint"/>
     </joint>
     <link name="robotiq_85_left_knuckle_link">
@@ -128,5 +127,4 @@
       <origin xyz="0.06142 0.0127 0" rpy="3.14 0.0 0.0" />
       <limit lower="-3.14" upper="3.14" velocity="3.14" effort="0.1"/>
-      <mimic joint="robotiq_85_left_knuckle_joint" offset="0"/>
     </joint>
     <joint name="robotiq_85_right_inner_knuckle_joint" type="revolute">
@@ -136,5 +134,4 @@
       <origin xyz="0.06142 -0.0127 0" rpy="0 0 0"/>
       <limit lower="-3.14" upper="3.14" velocity="3.14" effort="0.1"/>
-      <mimic joint="robotiq_85_left_knuckle_joint" offset="0"/>
     </joint>
     <link name="robotiq_85_left_inner_knuckle_link">
@@ -182,5 +179,4 @@
       <origin xyz="0.04303959807 -0.03759940821 0.0" rpy="0.0 0.0 0.0"/>
       <limit lower="-3.14" upper="3.14" velocity="3.14" effort="0.1"/>
-      <mimic joint="robotiq_85_left_knuckle_joint" multiplier="-1"/>
     </joint>
     <joint name="robotiq_85_right_finger_tip_joint" type="revolute">
@@ -190,5 +186,4 @@
       <origin rpy="0.0 0.0 0.0" xyz="0.04303959807 -0.03759940821  0.0"/>
       <limit lower="-3.14" upper="3.14" velocity="3.14" effort="0.1"/>
-      <mimic joint="robotiq_85_left_knuckle_joint" multiplier="-1"/>
     </joint>
     <link name="robotiq_85_left_finger_tip_link">

File: urdf/ur.ros2_control.xacro (robot description, xacro)
@@ -24,4 +24,5 @@
     <ros2_control name="${name}" type="system">
       <hardware>
+        <plugin>gz_ros2_control/GazeboSimSystem</plugin>
         <xacro:if value="${sim_gazebo}">
           <plugin>gazebo_ros2_control/GazeboSystem</plugin>
@@ -346,4 +347,63 @@
         <state_interface name="velocity"/>
       </joint>
+      <joint name="robotiq_85_left_inner_knuckle_joint">
+        <param name="mimic">robotiq_85_left_knuckle_joint</param>
+        <param name="offset">0.0</param>
+        <command_interface name="position"/>
+        <state_interface name="position">
+          <param name="initial_value">${initial_positions['robotiq_85_left_knuckle_joint']}</param>
+        </state_interface>
+        <state_interface name="velocity"/>
+      </joint>
+      <joint name="robotiq_85_left_finger_joint">
+        <command_interface name="position"/>
+        <state_interface name="position">
+          <param name="initial_value">${initial_positions['robotiq_85_left_knuckle_joint']}</param>
+        </state_interface>
+        <state_interface name="velocity"/>
+      </joint>
+      <joint name="robotiq_85_left_finger_tip_joint">
+        <param name="mimic">robotiq_85_left_knuckle_joint</param>
+        <param name="multiplier">-1.0</param>
+        <command_interface name="position"/>
+        <state_interface name="position">
+          <param name="initial_value">${initial_positions['robotiq_85_left_knuckle_joint']}</param>
+        </state_interface>
+        <state_interface name="velocity"/>
+      </joint>
+      <joint name="robotiq_85_right_knuckle_joint">
+        <param name="mimic">robotiq_85_left_knuckle_joint</param>
+        <param name="multiplier">1.0</param>
+        <command_interface name="position"/>
+        <state_interface name="position">
+          <param name="initial_value">${initial_positions['robotiq_85_left_knuckle_joint']}</param>
+        </state_interface>
+        <state_interface name="velocity"/>
+      </joint>
+      <joint name="robotiq_85_right_inner_knuckle_joint">
+        <param name="mimic">robotiq_85_left_knuckle_joint</param>
+        <param name="offset">0.0</param>
+        <command_interface name="position"/>
+        <state_interface name="position">
+          <param name="initial_value">${initial_positions['robotiq_85_left_knuckle_joint']}</param>
+        </state_interface>
+        <state_interface name="velocity"/>
+      </joint>
+      <joint name="robotiq_85_right_finger_joint">
+        <command_interface name="position"/>
+        <state_interface name="position">
+          <param name="initial_value">${initial_positions['robotiq_85_left_knuckle_joint']}</param>
+        </state_interface>
+        <state_interface name="velocity"/>
+      </joint>
+      <joint name="robotiq_85_right_finger_tip_joint">
+        <param name="mimic">robotiq_85_left_knuckle_joint</param>
+        <param name="multiplier">-1.0</param>
+        <command_interface name="position"/>
+        <state_interface name="position">
+          <param name="initial_value">${initial_positions['robotiq_85_left_knuckle_joint']}</param>
+        </state_interface>
+        <state_interface name="velocity"/>
+      </joint>
     </ros2_control>
   </xacro:macro>

File: urdf/ur.urdf.xacro (robot description, xacro)
@@ -138,3 +138,9 @@
     </gazebo>
   </xacro:if>
+  <gazebo>
+    <plugin filename="gz_ros2_control-system" name="gz_ros2_control::GazeboSimROS2ControlPlugin">
+      <robot_param>robot_description</robot_param>
+      <robot_param_node>robot_state_publisher</robot_param_node>
+    </plugin>
+  </gazebo>
 </robot>

File: urdf/ur_macro.xacro (robot description, xacro)
@@ -460,6 +460,6 @@
         <origin xyz="0.0 0.0 0.0" />
         <inertia ixx = "0.000380" ixy = "0.000000" ixz = "0.000000"
-             iyx = "0.000000" iyy = "0.001110" iyz = "0.000000"
-             izx = "0.000000" izy = "0.000000" izz = "0.001171" />
+             iyy = "0.001110" iyz = "0.000000"
+             izz = "0.001171" />
       </inertial>
     </link>
@@ -494,6 +494,6 @@
         <origin xyz="0.0 0.0 0.0" />
         <inertia ixx = "0.000009" ixy = "-0.000001" ixz = "0.000000"
-             iyx = "-0.000001" iyy = "0.000001" iyz = "0.000000"
-             izx = "0.000000" izy = "0.000000" izz = "0.000010" />
+             iyy = "0.000001" iyz = "0.000000"
+             izz = "0.000010" />
       </inertial>
     </link>
@@ -513,6 +513,6 @@
         <origin xyz="0.0 0.0 0.0" />
         <inertia ixx = "0.000009" ixy = "-0.000001" ixz = "0.000000"
-             iyx = "-0.000001" iyy = "0.000001" iyz = "0.000000"
-             izx = "0.000000" izy = "0.000000" izz = "0.000010" />
+             iyy = "0.000001" iyz = "0.000000"
+             izz = "0.000010" />
       </inertial>
     </link>
@@ -542,6 +542,6 @@
         <origin xyz="0.0 0.0 0.0" />
         <inertia ixx = "0.000003" ixy = "-0.000002" ixz = "0.000000"
-             iyx = "-0.000002" iyy = "0.000021" iyz = "0.000000"
-             izx = "0.000000" izy = "0.000000" izz = "0.000020" />
+             iyy = "0.000021" iyz = "0.000000"
+             izz = "0.000020" />
       </inertial>
     </link>
@@ -561,6 +561,6 @@
         <origin xyz="0.0 0.0 0.0" />
         <inertia ixx = "0.000003" ixy = "-0.000002" ixz = "0.000000"
-             iyx = "-0.000002" iyy = "0.000021" iyz = "0.000000"
-             izx = "0.000000" izy = "0.000000" izz = "0.000020" />
+             iyy = "0.000021" iyz = "0.000000"
+             izz = "0.000020" />
       </inertial>
     </link>
@@ -615,6 +615,6 @@
         <origin xyz="0.0 0.0 0.0" />
         <inertia ixx = "0.000039" ixy = "0.000000" ixz = "0.000000"
-             iyx = "0.000000" iyy = "0.000005" iyz = "0.000000"
-             izx = "0.000000" izy = "0.000000" izz = "0.000035" />
+             iyy = "0.000005" iyz = "0.000000"
+             izz = "0.000035" />
       </inertial>
     </link>
@@ -650,6 +650,6 @@
         <origin xyz="0.0 0.0 0.0" />
         <inertia ixx = "0.000002" ixy = "0.000000" ixz = "0.000000"
-             iyx = "0.000000" iyy = "0.000005" iyz = "0.000000"
-             izx = "0.000000" izy = "0.000000" izz = "0.000006" />
+             iyy = "0.000005" iyz = "0.000000"
+             izz = "0.000006" />
       </inertial>
     </link>
@@ -669,6 +669,6 @@
         <origin xyz="0.0 0.0 0.0" />
         <inertia ixx = "0.000002" ixy = "0.000000" ixz = "0.000000"
-             iyx = "0.000000" iyy = "0.000005" iyz = "0.000000"
-             izx = "0.000000" izy = "0.000000" izz = "0.000006" />
+             iyy = "0.000005" iyz = "0.000000"
+             izz = "0.000006" />
       </inertial>
     </link>

Commit message: Fix gripper bug (FINALLY)

File: urdf/gripper.urdf.xacro (robot description, xacro)
@@ -34,4 +34,5 @@
       <origin rpy="0.0 0.0 0.0" xyz="0.05490451627 -0.03060114443 0.0"/>
       <limit lower="-3.14" upper="3.14" velocity="3.14" effort="1000"/>
+      <mimic joint="robotiq_85_left_knuckle_joint" multiplier="1.0"/>
     </joint>
     <link name="robotiq_85_left_knuckle_link">
@@ -127,4 +128,5 @@
       <origin xyz="0.06142 0.0127 0" rpy="3.14 0.0 0.0" />
       <limit lower="-3.14" upper="3.14" velocity="3.14" effort="0.1"/>
+      <mimic joint="robotiq_85_left_knuckle_joint" offset="0.0"/>
     </joint>
     <joint name="robotiq_85_right_inner_knuckle_joint" type="revolute">
@@ -134,4 +136,5 @@
       <origin xyz="0.06142 -0.0127 0" rpy="0 0 0"/>
       <limit lower="-3.14" upper="3.14" velocity="3.14" effort="0.1"/>
+      <mimic joint="robotiq_85_left_knuckle_joint" offset="0.0"/>
     </joint>
     <link name="robotiq_85_left_inner_knuckle_link">
@@ -179,4 +182,5 @@
       <origin xyz="0.04303959807 -0.03759940821 0.0" rpy="0.0 0.0 0.0"/>
       <limit lower="-3.14" upper="3.14" velocity="3.14" effort="0.1"/>
+      <mimic joint="robotiq_85_left_knuckle_joint" multiplier="-1"/>
     </joint>
     <joint name="robotiq_85_right_finger_tip_joint" type="revolute">
@@ -186,4 +190,5 @@
       <origin rpy="0.0 0.0 0.0" xyz="0.04303959807 -0.03759940821  0.0"/>
       <limit lower="-3.14" upper="3.14" velocity="3.14" effort="0.1"/>
+      <mimic joint="robotiq_85_left_knuckle_joint" multiplier="-1"/>
     </joint>
     <link name="robotiq_85_left_finger_tip_link">

File: urdf/ur_macro.xacro (robot description, xacro)
@@ -469,5 +469,5 @@
       <axis xyz="0 0 1"/>
       <origin rpy="3.14 0.0 0.0" xyz="0.05490451627 0.03060114443 0.0"/>
-      <limit lower="0.0" upper="0.80285" velocity="3.14" effort="1000"/>
+      <limit lower="-0.1" upper="0.80285" velocity="3.14" effort="1000"/>
     </joint>
     <joint name="robotiq_85_right_knuckle_joint" type="revolute">
@@ -477,5 +477,6 @@
       <origin rpy="0.0 0.0 0.0" xyz="0.05490451627 -0.03060114443 0.0"/>
       <limit lower="-3.14" upper="3.14" velocity="3.14" effort="1000"/>
-      <mimic joint="robotiq_85_left_knuckle_joint"/>
+      <!-- <limit lower="-0.1" upper="0.80285" velocity="3.14" effort="1000"/> -->
+      <mimic joint="robotiq_85_left_knuckle_joint" multiplier="1.0"/>
     </joint>
     <link name="robotiq_85_left_knuckle_link">
@@ -493,5 +494,5 @@
         <mass value="0.018491" />
         <origin xyz="0.0 0.0 0.0" />
-        <inertia ixx = "0.000009" ixy = "-0.000001" ixz = "0.000000"
+        <inertia ixx = "0.000009" ixy = "0.000001" ixz = "0.000000"
              iyy = "0.000001" iyz = "0.000000"
              izz = "0.000010" />
@@ -512,5 +513,5 @@
         <mass value="0.018491" />
         <origin xyz="0.0 0.0 0.0" />
-        <inertia ixx = "0.000009" ixy = "-0.000001" ixz = "0.000000"
+        <inertia ixx = "0.000009" ixy = "0.000001" ixz = "0.000000"
              iyy = "0.000001" iyz = "0.000000"
              izz = "0.000010" />
@@ -541,5 +542,5 @@
         <mass value="0.027309" />
         <origin xyz="0.0 0.0 0.0" />
-        <inertia ixx = "0.000003" ixy = "-0.000002" ixz = "0.000000"
+        <inertia ixx = "0.000003" ixy = "0.000002" ixz = "0.000000"
              iyy = "0.000021" iyz = "0.000000"
              izz = "0.000020" />
@@ -560,5 +561,5 @@
         <mass value="0.027309" />
         <origin xyz="0.0 0.0 0.0" />
-        <inertia ixx = "0.000003" ixy = "-0.000002" ixz = "0.000000"
+        <inertia ixx = "0.000003" ixy = "0.000002" ixz = "0.000000"
              iyy = "0.000021" iyz = "0.000000"
              izz = "0.000020" />
@@ -570,4 +571,5 @@
       <axis xyz="0 0 1"/>
       <origin xyz="0.06142 0.0127 0" rpy="3.14 0.0 0.0" />
+      <!-- <limit lower="-0.1" upper="0.80285" velocity="3.14" effort="0.1"/> -->
       <limit lower="-3.14" upper="3.14" velocity="3.14" effort="0.1"/>
       <mimic joint="robotiq_85_left_knuckle_joint" offset="0"/>
@@ -578,4 +580,5 @@
       <axis xyz="0 0 1"/>
       <origin xyz="0.06142 -0.0127 0" rpy="0 0 0"/>
+      <!-- <limit lower="-0.1" upper="0.80285" velocity="3.14" effort="0.1"/> -->
       <limit lower="-3.14" upper="3.14" velocity="3.14" effort="0.1"/>
       <mimic joint="robotiq_85_left_knuckle_joint" offset="0"/>
@@ -596,6 +599,6 @@
         <origin xyz="0.0 0.0 0.0" />
         <inertia ixx = "0.000039" ixy = "0.000000" ixz = "0.000000"
-             iyx = "0.000000" iyy = "0.000005" iyz = "0.000000"
-             izx = "0.000000" izy = "0.000000" izz = "0.000035" />
+             iyy = "0.000005" iyz = "0.000000"
+             izz = "0.000035" />
       </inertial>
     </link>
@@ -624,4 +627,5 @@
       <axis xyz="0 0 1"/>
       <origin xyz="0.04303959807 -0.03759940821 0.0" rpy="0.0 0.0 0.0"/>
+      <!-- <limit lower="-0.80285" upper="0.1" velocity="3.14" effort="0.1"/> -->
       <limit lower="-3.14" upper="3.14" velocity="3.14" effort="0.1"/>
       <mimic joint="robotiq_85_left_knuckle_joint" multiplier="-1"/>
@@ -632,4 +636,5 @@
       <axis xyz="0 0 1"/>
       <origin rpy="0.0 0.0 0.0" xyz="0.04303959807 -0.03759940821  0.0"/>
+      <!-- <limit lower="-0.80285" upper="0.1" velocity="3.14" effort="0.1"/> -->
       <limit lower="-3.14" upper="3.14" velocity="3.14" effort="0.1"/>
       <mimic joint="robotiq_85_left_knuckle_joint" multiplier="-1"/>
