Commit message: Seperate gripper xacro file

File: urdf/gripper.urdf.xacro (robot description, xacro)
@@ -1,232 +1,275 @@
 <?xml version="1.0"?>
 <robot xmlns:xacro="http://www.ros.org/wiki/xacro" name="gripper">
-    <!-- Gripper -->
-    <link name="robotiq_85_base_link">
-      <visual>
-        <geometry>
-          <mesh filename="file://$(find my_ur)/meshes/robotiq_85_gripper/visual/robotiq_85_base_link.dae"/>
-        </geometry>
-      </visual>
-      <collision>
-        <geometry>
-          <mesh filename="file://$(find my_ur)/meshes/robotiq_85_gripper/collision/robotiq_85_base_link.stl"/>
-        </geometry>
-      </collision>
-      <inertial>
-        <mass value="0.636951" />
-        <origin xyz="0.0 0.0 0.0" />
-        <inertia ixx = "0.000380" ixy = "0.000000" ixz = "0.000000"
-             iyx = "0.000000" iyy = "0.001110" iyz = "0.000000"
-             izx = "0.000000" izy = "0.000000" izz = "0.001171" />
-      </inertial>
-    </link>
-    <joint name="robotiq_85_left_knuckle_joint" type="revolute">
-      <parent link="robotiq_85_base_link"/>
-      <child link="robotiq_85_left_knuckle_link"/>
-      <axis xyz="0 0 1"/>
-      <origin rpy="3.14 0.0 0.0" xyz="0.05490451627 0.03060114443 0.0"/>
-      <limit lower="0.0" upper="0.80285" velocity="3.14" effort="1000"/>
-    </joint>
-    <joint name="robotiq_85_right_knuckle_joint" type="revolute">
-      <parent link="robotiq_85_base_link"/>
-      <child link="robotiq_85_right_knuckle_link"/>
-      <axis xyz="0 0 1"/>
-      <origin rpy="0.0 0.0 0.0" xyz="0.05490451627 -0.03060114443 0.0"/>
-      <limit lower="-3.14" upper="3.14" velocity="3.14" effort="1000"/>
-      <mimic joint="robotiq_85_left_knuckle_joint" multiplier="1.0"/>
-    </joint>
-    <link name="robotiq_85_left_knuckle_link">
-      <visual>
-        <geometry>
-          <mesh filename="file://$(find my_ur)/meshes/robotiq_85_gripper/visual/robotiq_85_knuckle_link.dae"/>
-        </geometry>
-      </visual>
-      <collision>
-        <geometry>
-          <mesh filename="file://$(find my_ur)/meshes/robotiq_85_gripper/collision/robotiq_85_knuckle_link.stl"/>
-        </geometry>
-      </collision>
-      <inertial>
-        <mass value="0.018491" />
-        <origin xyz="0.0 0.0 0.0" />
-        <inertia ixx = "0.000009" ixy = "-0.000001" ixz = "0.000000"
-             iyx = "-0.000001" iyy = "0.000001" iyz = "0.000000"
-             izx = "0.000000" izy = "0.000000" izz = "0.000010" />
-      </inertial>
-    </link>
-    <link name="robotiq_85_right_knuckle_link">
-      <visual>
-        <geometry>
-          <mesh filename="file://$(find my_ur)/meshes/robotiq_85_gripper/visual/robotiq_85_knuckle_link.dae"/>
-        </geometry>
-      </visual>
-      <collision>
-        <geometry>
-          <mesh filename="file://$(find my_ur)/meshes/robotiq_85_gripper/collision/robotiq_85_knuckle_link.stl"/>
-        </geometry>
-      </collision>
-      <inertial>
-        <mass value="0.018491" />
-        <origin xyz="0.0 0.0 0.0" />
-        <inertia ixx = "0.000009" ixy = "-0.000001" ixz = "0.000000"
-             iyx = "-0.000001" iyy = "0.000001" iyz = "0.000000"
-             izx = "0.000000" izy = "0.000000" izz = "0.000010" />
-      </inertial>
-    </link>
-    <joint name="robotiq_85_left_finger_joint" type="fixed">
-      <parent link="robotiq_85_left_knuckle_link"/>
-      <child link="robotiq_85_left_finger_link"/>
-      <origin xyz="-0.00408552455 -0.03148604435 0.0" rpy="0 0 0" />
-    </joint>
-    <joint name="robotiq_85_right_finger_joint" type="fixed">
-      <parent link="robotiq_85_right_knuckle_link"/>
-      <child link="robotiq_85_right_finger_link"/>
-      <origin xyz="-0.00408552455 -0.03148604435 0.0" rpy="0 0 0" />
-    </joint>
-    <link name="robotiq_85_left_finger_link">
-      <visual>
-        <geometry>
-          <mesh filename="file://$(find my_ur)/meshes/robotiq_85_gripper/visual/robotiq_85_finger_link.dae"/>
-        </geometry>
-      </visual>
-      <collision>
-        <geometry>
-          <mesh filename="file://$(find my_ur)/meshes/robotiq_85_gripper/collision/robotiq_85_finger_link.stl"/>
-        </geometry>
-      </collision>
-      <inertial>
-        <mass value="0.027309" />
-        <origin xyz="0.0 0.0 0.0" />
-        <inertia ixx = "0.000003" ixy = "-0.000002" ixz = "0.000000"
-             iyx = "-0.000002" iyy = "0.000021" iyz = "0.000000"
-             izx = "0.000000" izy = "0.000000" izz = "0.000020" />
-      </inertial>
-    </link>
-    <link name="robotiq_85_right_finger_link">
-      <visual>
-        <geometry>
-          <mesh filename="file://$(find my_ur)/meshes/robotiq_85_gripper/visual/robotiq_85_finger_link.dae"/>
-        </geometry>
-      </visual>
-      <collision>
-        <geometry>
-          <mesh filename="file://$(find my_ur)/meshes/robotiq_85_gripper/collision/robotiq_85_finger_link.stl"/>
-        </geometry>
-      </collision>
-      <inertial>
-        <mass value="0.027309" />
-        <origin xyz="0.0 0.0 0.0" />
-        <inertia ixx = "0.000003" ixy = "-0.000002" ixz = "0.000000"
-             iyx = "-0.000002" iyy = "0.000021" iyz = "0.000000"
-             izx = "0.000000" izy = "0.000000" izz = "0.000020" />
-      </inertial>
-    </link>
-    <joint name="robotiq_85_left_inner_knuckle_joint" type="revolute">
-      <parent link="robotiq_85_base_link"/>
-      <child link="robotiq_85_left_inner_knuckle_link"/>
-      <axis xyz="0 0 1"/>
-      <origin xyz="0.06142 0.0127 0" rpy="3.14 0.0 0.0" />
-      <limit lower="-3.14" upper="3.14" velocity="3.14" effort="0.1"/>
-      <mimic joint="robotiq_85_left_knuckle_joint" offset="0.0"/>
-    </joint>
-    <joint name="robotiq_85_right_inner_knuckle_joint" type="revolute">
-      <parent link="robotiq_85_base_link"/>
-      <child link="robotiq_85_right_inner_knuckle_link"/>
-      <axis xyz="0 0 1"/>
-      <origin xyz="0.06142 -0.0127 0" rpy="0 0 0"/>
-      <limit lower="-3.14" upper="3.14" velocity="3.14" effort="0.1"/>
-      <mimic joint="robotiq_85_left_knuckle_joint" offset="0.0"/>
-    </joint>
-    <link name="robotiq_85_left_inner_knuckle_link">
-      <visual>
-        <geometry>
-          <mesh filename="file://$(find my_ur)/meshes/robotiq_85_gripper/visual/robotiq_85_inner_knuckle_link.dae"/>
-        </geometry>
-      </visual>
-      <collision>
-        <geometry>
-          <mesh filename="file://$(find my_ur)/meshes/robotiq_85_gripper/collision/robotiq_85_inner_knuckle_link.stl"/>
-        </geometry>
-      </collision>
-      <inertial>
-        <mass value="0.029951" />
-        <origin xyz="0.0 0.0 0.0" />
-        <inertia ixx = "0.000039" ixy = "0.000000" ixz = "0.000000"
-             iyx = "0.000000" iyy = "0.000005" iyz = "0.000000"
-             izx = "0.000000" izy = "0.000000" izz = "0.000035" />
-      </inertial>
-    </link>
-    <link name="robotiq_85_right_inner_knuckle_link">
-      <visual>
-        <geometry>
-          <mesh filename="file://$(find my_ur)/meshes/robotiq_85_gripper/visual/robotiq_85_inner_knuckle_link.dae"/>
-        </geometry>
-      </visual>
-      <collision>
-        <geometry>
-          <mesh filename="file://$(find my_ur)/meshes/robotiq_85_gripper/collision/robotiq_85_inner_knuckle_link.stl"/>
-        </geometry>
-      </collision>
-      <inertial>
-        <mass value="0.029951" />
-        <origin xyz="0.0 0.0 0.0" />
-        <inertia ixx = "0.000039" ixy = "0.000000" ixz = "0.000000"
-             iyx = "0.000000" iyy = "0.000005" iyz = "0.000000"
-             izx = "0.000000" izy = "0.000000" izz = "0.000035" />
-      </inertial>
-    </link>
-    <joint name="robotiq_85_left_finger_tip_joint" type="revolute">
-      <parent link="robotiq_85_left_inner_knuckle_link"/>
-      <child link="robotiq_85_left_finger_tip_link"/>
-      <axis xyz="0 0 1"/>
-      <origin xyz="0.04303959807 -0.03759940821 0.0" rpy="0.0 0.0 0.0"/>
-      <limit lower="-3.14" upper="3.14" velocity="3.14" effort="0.1"/>
-      <mimic joint="robotiq_85_left_knuckle_joint" multiplier="-1"/>
-    </joint>
-    <joint name="robotiq_85_right_finger_tip_joint" type="revolute">
-      <parent link="robotiq_85_right_inner_knuckle_link"/>
-      <child link="robotiq_85_right_finger_tip_link"/>
-      <axis xyz="0 0 1"/>
-      <origin rpy="0.0 0.0 0.0" xyz="0.04303959807 -0.03759940821  0.0"/>
-      <limit lower="-3.14" upper="3.14" velocity="3.14" effort="0.1"/>
-      <mimic joint="robotiq_85_left_knuckle_joint" multiplier="-1"/>
-    </joint>
-    <link name="robotiq_85_left_finger_tip_link">
-      <visual>
-        <geometry>
-          <mesh filename="file://$(find my_ur)/meshes/robotiq_85_gripper/visual/robotiq_85_finger_tip_link.dae"/>
-        </geometry>
-      </visual>
-      <collision>
-        <geometry>
-          <mesh filename="file://$(find my_ur)/meshes/robotiq_85_gripper/collision/robotiq_85_finger_tip_link.stl"/>
-        </geometry>
-      </collision>
-      <inertial>
-        <mass value="0.019555" />
-        <origin xyz="0.0 0.0 0.0" />
-        <inertia ixx = "0.000002" ixy = "0.000000" ixz = "0.000000"
-             iyx = "0.000000" iyy = "0.000005" iyz = "0.000000"
-             izx = "0.000000" izy = "0.000000" izz = "0.000006" />
-      </inertial>
-    </link>
-    <link name="robotiq_85_right_finger_tip_link">
-      <visual>
-        <geometry>
-          <mesh filename="file://$(find my_ur)/meshes/robotiq_85_gripper/visual/robotiq_85_finger_tip_link.dae"/>
-        </geometry>
-      </visual>
-      <collision>
-        <geometry>
-          <mesh filename="file://$(find my_ur)/meshes/robotiq_85_gripper/collision/robotiq_85_finger_tip_link.stl"/>
-        </geometry>
-      </collision>
-      <inertial>
-        <mass value="0.019555" />
-        <origin xyz="0.0 0.0 0.0" />
-        <inertia ixx = "0.000002" ixy = "0.000000" ixz = "0.000000"
-             iyx = "0.000000" iyy = "0.000005" iyz = "0.000000"
-             izx = "0.000000" izy = "0.000000" izz = "0.000006" />
-      </inertial>
-    </link>
+  <!-- Gripper -->
+  <link name="robotiq_85_base_link">
+    <visual>
+      <geometry>
+        <mesh filename="file://$(find my_ur)/meshes/robotiq_85_gripper/visual/robotiq_85_base_link.dae"/>
+      </geometry>
+    </visual>
+    <collision>
+      <geometry>
+        <mesh filename="file://$(find my_ur)/meshes/robotiq_85_gripper/collision/robotiq_85_base_link.stl"/>
+      </geometry>
+    </collision>
+    <inertial>
+      <mass value="0.636951" />
+      <origin xyz="0.0 0.0 0.0" />
+      <inertia ixx = "0.000380" ixy = "0.000000" ixz = "0.000000"
+          iyy = "0.001110" iyz = "0.000000"
+          izz = "0.001171" />
+    </inertial>
+  </link>
+  <joint name="robotiq_85_left_knuckle_joint" type="revolute">
+    <parent link="robotiq_85_base_link"/>
+    <child link="robotiq_85_left_knuckle_link"/>
+    <axis xyz="0 0 1"/>
+    <origin rpy="3.14 0.0 0.0" xyz="0.05490451627 0.03060114443 0.0"/>
+    <limit lower="-0.1" upper="0.80285" velocity="3.14" effort="1000"/>
+  </joint>
+  <joint name="robotiq_85_right_knuckle_joint" type="revolute">
+    <parent link="robotiq_85_base_link"/>
+    <child link="robotiq_85_right_knuckle_link"/>
+    <axis xyz="0 0 1"/>
+    <origin rpy="0.0 0.0 0.0" xyz="0.05490451627 -0.03060114443 0.0"/>
+    <limit lower="-3.14" upper="3.14" velocity="3.14" effort="1000"/>
+    <!-- <limit lower="-0.1" upper="0.80285" velocity="3.14" effort="1000"/> -->
+    <mimic joint="robotiq_85_left_knuckle_joint" multiplier="1.0"/>
+  </joint>
+  <link name="robotiq_85_left_knuckle_link">
+    <visual>
+      <geometry>
+        <mesh filename="file://$(find my_ur)/meshes/robotiq_85_gripper/visual/robotiq_85_knuckle_link.dae"/>
+      </geometry>
+    </visual>
+    <collision>
+      <geometry>
+        <mesh filename="file://$(find my_ur)/meshes/robotiq_85_gripper/collision/robotiq_85_knuckle_link.stl"/>
+      </geometry>
+    </collision>
+    <inertial>
+      <mass value="0.018491" />
+      <origin xyz="0.0 0.0 0.0" />
+      <inertia ixx = "0.000009" ixy = "0.000001" ixz = "0.000000"
+          iyy = "0.000001" iyz = "0.000000"
+          izz = "0.000010" />
+    </inertial>
+  </link>
+  <link name="robotiq_85_right_knuckle_link">
+    <visual>
+      <geometry>
+        <mesh filename="file://$(find my_ur)/meshes/robotiq_85_gripper/visual/robotiq_85_knuckle_link.dae"/>
+      </geometry>
+    </visual>
+    <collision>
+      <geometry>
+        <mesh filename="file://$(find my_ur)/meshes/robotiq_85_gripper/collision/robotiq_85_knuckle_link.stl"/>
+      </geometry>
+    </collision>
+    <inertial>
+      <mass value="0.018491" />
+      <origin xyz="0.0 0.0 0.0" />
+      <inertia ixx = "0.000009" ixy = "0.000001" ixz = "0.000000"
+          iyy = "0.000001" iyz = "0.000000"
+          izz = "0.000010" />
+    </inertial>
+  </link>
+  <joint name="robotiq_85_left_finger_joint" type="fixed">
+    <parent link="robotiq_85_left_knuckle_link"/>
+    <child link="robotiq_85_left_finger_link"/>
+    <origin xyz="-0.00408552455 -0.03148604435 0.0" rpy="0 0 0" />
+  </joint>
+  <joint name="robotiq_85_right_finger_joint" type="fixed">
+    <parent link="robotiq_85_right_knuckle_link"/>
+    <child link="robotiq_85_right_finger_link"/>
+    <origin xyz="-0.00408552455 -0.03148604435 0.0" rpy="0 0 0" />
+  </joint>
+  <link name="robotiq_85_left_finger_link">
+    <visual>
+      <geometry>
+        <mesh filename="file://$(find my_ur)/meshes/robotiq_85_gripper/visual/robotiq_85_finger_link.dae"/>
+      </geometry>
+    </visual>
+    <collision>
+      <geometry>
+        <mesh filename="file://$(find my_ur)/meshes/robotiq_85_gripper/collision/robotiq_85_finger_link.stl"/>
+      </geometry>
+      <surface>
+        <friction>
+          <ode>
+            <mu>100.0</mu>
+            <mu2>100.0</mu2>
+          </ode>
+        </friction>
+        <contact>
+          <ode>
+            <kp>10000.0</kp>
+            <kd>1.0</kd>
+            <max_vel>0.1</max_vel>
+            <min_depth>0.001</min_depth>
+          </ode>
+        </contact>
+      </surface>
+    </collision>
+    <inertial>
+      <mass value="0.027309" />
+      <origin xyz="0.0 0.0 0.0" />
+      <inertia ixx = "0.000003" ixy = "0.000002" ixz = "0.000000"
+          iyy = "0.000021" iyz = "0.000000"
+          izz = "0.000020" />
+    </inertial>
+  </link>
+  <link name="robotiq_85_right_finger_link">
+    <visual>
+      <geometry>
+        <mesh filename="file://$(find my_ur)/meshes/robotiq_85_gripper/visual/robotiq_85_finger_link.dae"/>
+      </geometry>
+    </visual>
+    <collision>
+      <geometry>
+        <mesh filename="file://$(find my_ur)/meshes/robotiq_85_gripper/collision/robotiq_85_finger_link.stl"/>
+      </geometry>
+      <surface>
+        <friction>
+          <ode>
+            <mu>100.0</mu>
+            <mu2>100.0</mu2>
+          </ode>
+        </friction>
+        <contact>
+          <ode>
+            <kp>10000.0</kp>
+            <kd>1.0</kd>
+            <max_vel>0.1</max_vel>
+            <min_depth>0.001</min_depth>
+          </ode>
+        </contact>
+      </surface>
+    </collision>
+    <inertial>
+      <mass value="0.027309" />
+      <origin xyz="0.0 0.0 0.0" />
+      <inertia ixx = "0.000003" ixy = "0.000002" ixz = "0.000000"
+          iyy = "0.000021" iyz = "0.000000"
+          izz = "0.000020" />
+    </inertial>
+  </link>
+  <joint name="robotiq_85_left_inner_knuckle_joint" type="revolute">
+    <parent link="robotiq_85_base_link"/>
+    <child link="robotiq_85_left_inner_knuckle_link"/>
+    <axis xyz="0 0 1"/>
+    <origin xyz="0.06142 0.0127 0" rpy="3.14 0.0 0.0" />
+    <!-- <limit lower="-0.1" upper="0.80285" velocity="3.14" effort="0.1"/> -->
+    <limit lower="-3.14" upper="3.14" velocity="3.14" effort="0.1"/>
+    <mimic joint="robotiq_85_left_knuckle_joint" offset="0"/>
+  </joint>
+  <joint name="robotiq_85_right_inner_knuckle_joint" type="revolute">
+    <parent link="robotiq_85_base_link"/>
+    <child link="robotiq_85_right_inner_knuckle_link"/>
+    <axis xyz="0 0 1"/>
+    <origin xyz="0.06142 -0.0127 0" rpy="0 0 0"/>
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