Commit message: Attach gripper to UR10 urdf

File: urdf/ur.ros2_control.xacro (robot description, xacro)
@@ -338,4 +338,61 @@
         </gpio>
       </xacro:unless>
+      <!-- Gripper Hardware Interface -->
+      <joint name="robotiq_85_left_knuckle_joint">
+        <command_interface name="position"/>
+        <command_interface name="velocity"/>
+        <state_interface name="position" />
+        <state_interface name="velocity"/>
+        <state_interface name="effort"/>
+      </joint>
+      <joint name="robotiq_85_left_finger_joint">
+        <command_interface name="position"/>
+        <command_interface name="velocity"/>
+        <state_interface name="position" />
+        <state_interface name="velocity"/>
+        <state_interface name="effort"/>
+      </joint>
+      <joint name="robotiq_85_left_inner_knuckle_joint">
+        <command_interface name="position"/>
+        <command_interface name="velocity"/>
+        <state_interface name="position" />
+        <state_interface name="velocity"/>
+        <state_interface name="effort"/>
+      </joint>
+      <joint name="robotiq_85_left_tip_joint">
+        <command_interface name="position"/>
+        <command_interface name="velocity"/>
+        <state_interface name="position" />
+        <state_interface name="velocity"/>
+        <state_interface name="effort"/>
+      </joint>
+      <joint name="robotiq_85_right_knuckle_joint">
+        <command_interface name="position"/>
+        <command_interface name="velocity"/>
+        <state_interface name="position" />
+        <state_interface name="velocity"/>
+        <state_interface name="effort"/>
+      </joint>
+      <joint name="robotiq_85_right_finger_joint">
+        <command_interface name="position"/>
+        <command_interface name="velocity"/>
+        <state_interface name="position" />
+        <state_interface name="velocity"/>
+        <state_interface name="effort"/>
+      </joint>
+      <joint name="robotiq_85_right_inner_knuckle_joint">
+        <command_interface name="position"/>
+        <command_interface name="velocity"/>
+        <state_interface name="position" />
+        <state_interface name="velocity"/>
+        <state_interface name="effort"/>
+      </joint>
+      <joint name="robotiq_85_right_tip_joint">
+        <command_interface name="position"/>
+        <command_interface name="velocity"/>
+        <state_interface name="position" />
+        <state_interface name="velocity"/>
+        <state_interface name="effort"/>
+      </joint>
     </ros2_control>
   </xacro:macro>

File: urdf/ur_macro.xacro (robot description, xacro)
@@ -444,4 +444,239 @@
       <child link="${tf_prefix}tool0"/>
     </joint>
+    <!-- Gripper -->
+    <link name="robotiq_85_base_link">
+      <visual>
+        <geometry>
+          <mesh filename="file://$(find my_ur)/meshes/robotiq_85_gripper/visual/robotiq_85_base_link.dae"/>
+        </geometry>
+      </visual>
+      <collision>
+        <geometry>
+          <mesh filename="file://$(find my_ur)/meshes/robotiq_85_gripper/collision/robotiq_85_base_link.stl"/>
+        </geometry>
+      </collision>
+      <inertial>
+        <mass value="0.636951" />
+        <origin xyz="0.0 0.0 0.0" />
+        <inertia ixx = "0.000380" ixy = "0.000000" ixz = "0.000000"
+             iyx = "0.000000" iyy = "0.001110" iyz = "0.000000"
+             izx = "0.000000" izy = "0.000000" izz = "0.001171" />
+      </inertial>
+    </link>
+    <joint name="robotiq_85_left_knuckle_joint" type="revolute">
+      <parent link="robotiq_85_base_link"/>
+      <child link="robotiq_85_left_knuckle_link"/>
+      <axis xyz="0 0 1"/>
+      <origin rpy="3.14 0.0 0.0" xyz="0.05490451627 0.03060114443 0.0"/>
+      <limit lower="0.0" upper="0.80285" velocity="3.14" effort="1000"/>
+    </joint>
+    <joint name="robotiq_85_right_knuckle_joint" type="revolute">
+      <parent link="robotiq_85_base_link"/>
+      <child link="robotiq_85_right_knuckle_link"/>
+      <axis xyz="0 0 1"/>
+      <origin rpy="0.0 0.0 0.0" xyz="0.05490451627 -0.03060114443 0.0"/>
+      <limit lower="-3.14" upper="3.14" velocity="3.14" effort="1000"/>
+      <mimic joint="robotiq_85_left_knuckle_joint"/>
+    </joint>
+    <link name="robotiq_85_left_knuckle_link">
+      <visual>
+        <geometry>
+          <mesh filename="file://$(find my_ur)/meshes/robotiq_85_gripper/visual/robotiq_85_knuckle_link.dae"/>
+        </geometry>
+      </visual>
+      <collision>
+        <geometry>
+          <mesh filename="file://$(find my_ur)/meshes/robotiq_85_gripper/collision/robotiq_85_knuckle_link.stl"/>
+        </geometry>
+      </collision>
+      <inertial>
+        <mass value="0.018491" />
+        <origin xyz="0.0 0.0 0.0" />
+        <inertia ixx = "0.000009" ixy = "-0.000001" ixz = "0.000000"
+             iyx = "-0.000001" iyy = "0.000001" iyz = "0.000000"
+             izx = "0.000000" izy = "0.000000" izz = "0.000010" />
+      </inertial>
+    </link>
+    <link name="robotiq_85_right_knuckle_link">
+      <visual>
+        <geometry>
+          <mesh filename="file://$(find my_ur)/meshes/robotiq_85_gripper/visual/robotiq_85_knuckle_link.dae"/>
+        </geometry>
+      </visual>
+      <collision>
+        <geometry>
+          <mesh filename="file://$(find my_ur)/meshes/robotiq_85_gripper/collision/robotiq_85_knuckle_link.stl"/>
+        </geometry>
+      </collision>
+      <inertial>
+        <mass value="0.018491" />
+        <origin xyz="0.0 0.0 0.0" />
+        <inertia ixx = "0.000009" ixy = "-0.000001" ixz = "0.000000"
+             iyx = "-0.000001" iyy = "0.000001" iyz = "0.000000"
+             izx = "0.000000" izy = "0.000000" izz = "0.000010" />
+      </inertial>
+    </link>
+    <joint name="robotiq_85_left_finger_joint" type="fixed">
+      <parent link="robotiq_85_left_knuckle_link"/>
+      <child link="robotiq_85_left_finger_link"/>
+      <origin xyz="-0.00408552455 -0.03148604435 0.0" rpy="0 0 0" />
+    </joint>
+    <joint name="robotiq_85_right_finger_joint" type="fixed">
+      <parent link="robotiq_85_right_knuckle_link"/>
+      <child link="robotiq_85_right_finger_link"/>
+      <origin xyz="-0.00408552455 -0.03148604435 0.0" rpy="0 0 0" />
+    </joint>
+    <link name="robotiq_85_left_finger_link">
+      <visual>
+        <geometry>
+          <mesh filename="file://$(find my_ur)/meshes/robotiq_85_gripper/visual/robotiq_85_finger_link.dae"/>
+        </geometry>
+      </visual>
+      <collision>
+        <geometry>
+          <mesh filename="file://$(find my_ur)/meshes/robotiq_85_gripper/collision/robotiq_85_finger_link.stl"/>
+        </geometry>
+      </collision>
+      <inertial>
+        <mass value="0.027309" />
+        <origin xyz="0.0 0.0 0.0" />
+        <inertia ixx = "0.000003" ixy = "-0.000002" ixz = "0.000000"
+             iyx = "-0.000002" iyy = "0.000021" iyz = "0.000000"
+             izx = "0.000000" izy = "0.000000" izz = "0.000020" />
+      </inertial>
+    </link>
+    <link name="robotiq_85_right_finger_link">
+      <visual>
+        <geometry>
+          <mesh filename="file://$(find my_ur)/meshes/robotiq_85_gripper/visual/robotiq_85_finger_link.dae"/>
+        </geometry>
+      </visual>
+      <collision>
+        <geometry>
+          <mesh filename="file://$(find my_ur)/meshes/robotiq_85_gripper/collision/robotiq_85_finger_link.stl"/>
+        </geometry>
+      </collision>
+      <inertial>
+        <mass value="0.027309" />
+        <origin xyz="0.0 0.0 0.0" />
+        <inertia ixx = "0.000003" ixy = "-0.000002" ixz = "0.000000"
+             iyx = "-0.000002" iyy = "0.000021" iyz = "0.000000"
+             izx = "0.000000" izy = "0.000000" izz = "0.000020" />
+      </inertial>
+    </link>
+    <joint name="robotiq_85_left_inner_knuckle_joint" type="revolute">
+      <parent link="robotiq_85_base_link"/>
+      <child link="robotiq_85_left_inner_knuckle_link"/>
+      <axis xyz="0 0 1"/>
+      <origin xyz="0.06142 0.0127 0" rpy="3.14 0.0 0.0" />
+      <limit lower="-3.14" upper="3.14" velocity="3.14" effort="0.1"/>
+      <mimic joint="robotiq_85_left_knuckle_joint" offset="0"/>
+    </joint>
+    <joint name="robotiq_85_right_inner_knuckle_joint" type="revolute">
+      <parent link="robotiq_85_base_link"/>
+      <child link="robotiq_85_right_inner_knuckle_link"/>
+      <axis xyz="0 0 1"/>
+      <origin xyz="0.06142 -0.0127 0" rpy="0 0 0"/>
+      <limit lower="-3.14" upper="3.14" velocity="3.14" effort="0.1"/>
+      <mimic joint="robotiq_85_left_knuckle_joint" offset="0"/>
+    </joint>
+    <link name="robotiq_85_left_inner_knuckle_link">
+      <visual>
+        <geometry>
+          <mesh filename="file://$(find my_ur)/meshes/robotiq_85_gripper/visual/robotiq_85_inner_knuckle_link.dae"/>
+        </geometry>
+      </visual>
+      <collision>
+        <geometry>
+          <mesh filename="file://$(find my_ur)/meshes/robotiq_85_gripper/collision/robotiq_85_inner_knuckle_link.stl"/>
+        </geometry>
+      </collision>
+      <inertial>
+        <mass value="0.029951" />
+        <origin xyz="0.0 0.0 0.0" />
+        <inertia ixx = "0.000039" ixy = "0.000000" ixz = "0.000000"
+             iyx = "0.000000" iyy = "0.000005" iyz = "0.000000"
+             izx = "0.000000" izy = "0.000000" izz = "0.000035" />
+      </inertial>
+    </link>
+    <link name="robotiq_85_right_inner_knuckle_link">
+      <visual>
+        <geometry>
+          <mesh filename="file://$(find my_ur)/meshes/robotiq_85_gripper/visual/robotiq_85_inner_knuckle_link.dae"/>
+        </geometry>
+      </visual>
+      <collision>
+        <geometry>
+          <mesh filename="file://$(find my_ur)/meshes/robotiq_85_gripper/collision/robotiq_85_inner_knuckle_link.stl"/>
+        </geometry>
+      </collision>
+      <inertial>
+        <mass value="0.029951" />
+        <origin xyz="0.0 0.0 0.0" />
+        <inertia ixx = "0.000039" ixy = "0.000000" ixz = "0.000000"
+             iyx = "0.000000" iyy = "0.000005" iyz = "0.000000"
+             izx = "0.000000" izy = "0.000000" izz = "0.000035" />
+      </inertial>
+    </link>
+    <joint name="robotiq_85_left_finger_tip_joint" type="revolute">
+      <parent link="robotiq_85_left_inner_knuckle_link"/>
+      <child link="robotiq_85_left_finger_tip_link"/>
+      <axis xyz="0 0 1"/>
+      <origin xyz="0.04303959807 -0.03759940821 0.0" rpy="0.0 0.0 0.0"/>
+      <limit lower="-3.14" upper="3.14" velocity="3.14" effort="0.1"/>
+      <mimic joint="robotiq_85_left_knuckle_joint" multiplier="-1"/>
+    </joint>
+    <joint name="robotiq_85_right_finger_tip_joint" type="revolute">
+      <parent link="robotiq_85_right_inner_knuckle_link"/>
+      <child link="robotiq_85_right_finger_tip_link"/>
+      <axis xyz="0 0 1"/>
+      <origin rpy="0.0 0.0 0.0" xyz="0.04303959807 -0.03759940821  0.0"/>
+      <limit lower="-3.14" upper="3.14" velocity="3.14" effort="0.1"/>
+      <mimic joint="robotiq_85_left_knuckle_joint" multiplier="-1"/>
+    </joint>
+    <link name="robotiq_85_left_finger_tip_link">
+      <visual>
+        <geometry>
+          <mesh filename="file://$(find my_ur)/meshes/robotiq_85_gripper/visual/robotiq_85_finger_tip_link.dae"/>
+        </geometry>
+      </visual>
+      <collision>
+        <geometry>
+          <mesh filename="file://$(find my_ur)/meshes/robotiq_85_gripper/collision/robotiq_85_finger_tip_link.stl"/>
+        </geometry>
+      </collision>
+      <inertial>
+        <mass value="0.019555" />
+        <origin xyz="0.0 0.0 0.0" />
+        <inertia ixx = "0.000002" ixy = "0.000000" ixz = "0.000000"
+             iyx = "0.000000" iyy = "0.000005" iyz = "0.000000"
+             izx = "0.000000" izy = "0.000000" izz = "0.000006" />
+      </inertial>
+    </link>
+    <link name="robotiq_85_right_finger_tip_link">
+      <visual>
+        <geometry>
+          <mesh filename="file://$(find my_ur)/meshes/robotiq_85_gripper/visual/robotiq_85_finger_tip_link.dae"/>
+        </geometry>
+      </visual>
+      <collision>
+        <geometry>
+          <mesh filename="file://$(find my_ur)/meshes/robotiq_85_gripper/collision/robotiq_85_finger_tip_link.stl"/>
+        </geometry>
+      </collision>
+      <inertial>
+        <mass value="0.019555" />
+        <origin xyz="0.0 0.0 0.0" />
+        <inertia ixx = "0.000002" ixy = "0.000000" ixz = "0.000000"
+             iyx = "0.000000" iyy = "0.000005" iyz = "0.000000"
+             izx = "0.000000" izy = "0.000000" izz = "0.000006" />
+      </inertial>
+    </link>
+    <!-- Connect gripper to arm -->
+    <joint name="arm_gripper_joint" type="fixed">
+      <parent link="${tf_prefix}wrist_3_link"/>
+      <child link="robotiq_85_base_link"/>
+      <origin rpy="0.0 -1.5708 0.0" xyz="0.0 0.0 0.0"/>
+    </joint>
   </xacro:macro>
 </robot>

Commit message: Allow Moveit to control gripper

File: urdf/ur.ros2_control.xacro (robot description, xacro)
@@ -7,5 +7,5 @@
     sim_ignition:=false
     headless_mode:=false
-    initial_positions:=${dict(shoulder_pan_joint=0.0,shoulder_lift_joint=-1.57,elbow_joint=0.0,wrist_1_joint=-1.57,wrist_2_joint=0.0,wrist_3_joint=0.0)}
+    initial_positions:=${dict(shoulder_pan_joint=0.0,shoulder_lift_joint=-1.57,elbow_joint=0.0,wrist_1_joint=-1.57,wrist_2_joint=0.0,wrist_3_joint=0.0, robotiq_85_left_knuckle_joint=0.0)}
     use_tool_communication:=false
     script_filename output_recipe_filename
@@ -341,57 +341,8 @@
       <joint name="robotiq_85_left_knuckle_joint">
         <command_interface name="position"/>
-        <command_interface name="velocity"/>
-        <state_interface name="position" />
-        <state_interface name="velocity"/>
-        <state_interface name="effort"/>
-      </joint>
-      <joint name="robotiq_85_left_finger_joint">
-        <command_interface name="position"/>
-        <command_interface name="velocity"/>
-        <state_interface name="position" />
-        <state_interface name="velocity"/>
-        <state_interface name="effort"/>
-      </joint>
-      <joint name="robotiq_85_left_inner_knuckle_joint">
-        <command_interface name="position"/>
-        <command_interface name="velocity"/>
-        <state_interface name="position" />
-        <state_interface name="velocity"/>
-        <state_interface name="effort"/>
-      </joint>
-      <joint name="robotiq_85_left_tip_joint">
-        <command_interface name="position"/>
-        <command_interface name="velocity"/>
-        <state_interface name="position" />
-        <state_interface name="velocity"/>
-        <state_interface name="effort"/>
-      </joint>
-      <joint name="robotiq_85_right_knuckle_joint">
-        <command_interface name="position"/>
-        <command_interface name="velocity"/>
-        <state_interface name="position" />
-        <state_interface name="velocity"/>
-        <state_interface name="effort"/>
-      </joint>
-      <joint name="robotiq_85_right_finger_joint">
-        <command_interface name="position"/>
-        <command_interface name="velocity"/>
-        <state_interface name="position" />
-        <state_interface name="velocity"/>
-        <state_interface name="effort"/>
-      </joint>
-      <joint name="robotiq_85_right_inner_knuckle_joint">
-        <command_interface name="position"/>
-        <command_interface name="velocity"/>
-        <state_interface name="position" />
-        <state_interface name="velocity"/>
-        <state_interface name="effort"/>
-      </joint>
-      <joint name="robotiq_85_right_tip_joint">
-        <command_interface name="position"/>
-        <command_interface name="velocity"/>
-        <state_interface name="position" />
-        <state_interface name="velocity"/>
-        <state_interface name="effort"/>
+        <state_interface name="position">
+          <param name="initial_value">${initial_positions['robotiq_85_left_knuckle_joint']}</param>
+        </state_interface>
+        <state_interface name="velocity"/>
       </joint>
     </ros2_control>

Commit message: Remove more gripper stuff, add sander

File: urdf/ur.ros2_control.xacro (robot description, xacro)
@@ -339,71 +339,4 @@
         </gpio>
       </xacro:unless>
-      <!-- Gripper Hardware Interface -->
-      <joint name="robotiq_85_left_knuckle_joint">
-        <command_interface name="position"/>
-        <state_interface name="position">
-          <param name="initial_value">${initial_positions['robotiq_85_left_knuckle_joint']}</param>
-        </state_interface>
-        <state_interface name="velocity"/>
-      </joint>
-      <joint name="robotiq_85_left_inner_knuckle_joint">
-        <param name="mimic">robotiq_85_left_knuckle_joint</param>
-        <param name="offset">0.0</param>
-        <command_interface name="position"/>
-        <state_interface name="position">
-          <param name="initial_value">${initial_positions['robotiq_85_left_knuckle_joint']}</param>
-        </state_interface>
-        <state_interface name="velocity"/>
-      </joint>
-      <joint name="robotiq_85_left_finger_joint">
-        <command_interface name="position"/>
-        <state_interface name="position">
-          <param name="initial_value">${initial_positions['robotiq_85_left_knuckle_joint']}</param>
-        </state_interface>
-        <state_interface name="velocity"/>
-      </joint>
-      <joint name="robotiq_85_left_finger_tip_joint">
-        <param name="mimic">robotiq_85_left_knuckle_joint</param>
-        <param name="multiplier">-1.0</param>
-        <command_interface name="position"/>
-        <state_interface name="position">
-          <param name="initial_value">${initial_positions['robotiq_85_left_knuckle_joint']}</param>
-        </state_interface>
-        <state_interface name="velocity"/>
-      </joint>
-      <joint name="robotiq_85_right_knuckle_joint">
-        <param name="mimic">robotiq_85_left_knuckle_joint</param>
-        <param name="multiplier">1.0</param>
-        <command_interface name="position"/>
-        <state_interface name="position">
-          <param name="initial_value">${initial_positions['robotiq_85_left_knuckle_joint']}</param>
-        </state_interface>
-        <state_interface name="velocity"/>
-      </joint>
-      <joint name="robotiq_85_right_inner_knuckle_joint">
-        <param name="mimic">robotiq_85_left_knuckle_joint</param>
-        <param name="offset">0.0</param>
-        <command_interface name="position"/>
-        <state_interface name="position">
-          <param name="initial_value">${initial_positions['robotiq_85_left_knuckle_joint']}</param>
-        </state_interface>
-        <state_interface name="velocity"/>
-      </joint>
-      <joint name="robotiq_85_right_finger_joint">
-        <command_interface name="position"/>
-        <state_interface name="position">
-          <param name="initial_value">${initial_positions['robotiq_85_left_knuckle_joint']}</param>
-        </state_interface>
-        <state_interface name="velocity"/>
-      </joint>
-      <joint name="robotiq_85_right_finger_tip_joint">
-        <param name="mimic">robotiq_85_left_knuckle_joint</param>
-        <param name="multiplier">-1.0</param>
-        <command_interface name="position"/>
-        <state_interface name="position">
-          <param name="initial_value">${initial_positions['robotiq_85_left_knuckle_joint']}</param>
-        </state_interface>
-        <state_interface name="velocity"/>
-      </joint>
     </ros2_control>
   </xacro:macro>

File: urdf/ur_macro.xacro (robot description, xacro)
@@ -444,6 +444,6 @@
       <child link="${tf_prefix}tool0"/>
     </joint>
-    <!-- Gripper URDF -->
-    <xacro:include filename="$(find my_ur)/urdf/gripper.urdf.xacro" />
+    <!-- Sander URDF -->
+    <xacro:include filename="$(find my_ur)/urdf/simple_sander.urdf.xacro" />
   </xacro:macro>
 </robot>
